File: keyboard/keyboard.kicad_pcb (KiCad board)
At the start: 2 copper layers, 189.9 x 143.3 mm, 69 parts, among them U1 Pico

Commit message: writing
Parts:
- moved H2 28.3 mm to (123.2, 87.6)
- moved H3 2.87 mm to (214.0, 87.6)
- moved H1 1.97 mm to (95.9, 27.3)
Connections:
- U1 pad 16: unconnected-(U1-GPIO12-Pad16) -> Row1
- U1 pad 17: Row1 -> Row2
- U1 pad 19: Row2 -> Row3
- U1 pad 20: Row3 -> unconnected-(U1-GPIO15-Pad20)
Routing:
- net Col7: track 160.0 -> 139.9 mm
- net Col6: track 191.2 -> 200.4 mm
- net Row2: track 142.2 -> 136.1 mm
- net Row1: track 163.2 -> 160.7 mm
- net Col4: track 142.1 -> 140.3 mm
- net Col5: track 184.1 -> 182.6 mm
- net Row3: track 134.0 -> 135.4 mm
Other:
- board size 189.9 x 143.3 mm -> 188.6 x 140.8 mm
